File: PCB/9DofImu.brd (EAGLE design)
At the start: 63.7 x 47.3 mm, 37 parts, among them U1 ATMEGA328, U2 ITG-3200, U3 LSM303

Commit message: upadted pcb
Parts:
- added JP3: FTDI Basic, SparkFun:1X06-SMD
Changed lines of the file:
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@@
 <setting verticaltext="up"/>
 </settings>
-<grid distance="0.0125" unitdist="inch" unit="inch" style="lines" multiple="1" display="yes" altdistance="0.000000123031" altunitdist="inch" altunit="inch"/>
+<grid distance="0.1" unitdist="inch" unit="inch" style="lines" multiple="1" display="yes" altdistance="0.000000123031" altunitdist="inch" altunit="inch"/>
 <layers>
 <layer number="1" name="Top" color="4" fill="1" visible="yes" active="yes"/>
@@
 <element name="JP2" library="SparkFun" package="1X06-SMD" value="FTDI Basic" x="72.314103125" y="33.453025" rot="R90"/>
 <element name="U$2" library="fab" package="SJFAB" value="SOLDER_JUMPER" x="15.5575" y="6.985" rot="R180"/>
+<element name="JP3" library="SparkFun" package="1X06-SMD" value="FTDI Basic" x="60.798259375" y="8.0344875" rot="R180"/>
 </elements>
 <signals>

Commit message: pcb updates
Parts:
- added J1, J2, J3, J4: (no value), SparkFun-Connectors:1X01NS-KIT
- JP1, JP2, JP3: device SparkFun:1X06-SMD -> SparkFun:1X06-KIT
- moved JP2 27.4 mm to (47.8, 45.6), turned to 180 degrees
- moved JP3 14.7 mm to (47.8, 15.1), turned to 270 degrees
- moved C1 7.62 mm to (35.4, 28.5)
- moved U2 7.62 mm to (27.1, 33.9)
- moved C15 7.62 mm to (27.9, 12.2)
- moved C4 7.62 mm to (21.2, 28.9)
- moved C5 7.62 mm to (25.8, 40.2)
- moved C6 7.62 mm to (29.6, 40.2)
- moved C8 7.62 mm to (22.8, 33.8)
- moved R10 7.62 mm to (23.6, 23.2)
- moved R11 7.62 mm to (23.6, 20.5)
- moved R12 7.62 mm to (31.1, 21.2)
- moved R13 7.62 mm to (20.1, 44.2)
- moved R4 7.62 mm to (26.9, 26.6)
- moved U$1 7.62 mm to (18.4, 6.50)
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Connections:
- net GND: now also J4.1, R1.2
- net MISO: now also J1.1
- net MOSI: now also J3.1
- net SCK: now also J2.1
Routing:
- net GND: track 264.0 -> 221.7 mm
- net MOSI: track 7.18 -> 9.52 mm
- net SCK: track 26.7 -> 24.8 mm
- net 3.3V: track 206.9 -> 205.2 mm
- added copper zone on layer 1, net GND
Other:
- board size 63.7 x 47.3 mm -> 55.9 x 54 mm

Commit message: i2c pin headers
Parts:
- removed J3, J4: (no value), SparkFun-Connectors:1X01NS-KIT
- J1, J2: device SparkFun-Connectors:1X01NS-KIT -> SparkFun-Connectors:1X01
- moved J1 25.3 mm to (34.9, 23.5)
- moved J2 19.0 mm to (34.9, 21.0)
Connections:
- net GND: no longer J4.1
- net MISO: no longer J1.1
- net MOSI: no longer J3.1
- net SCK: no longer J2.1
- net SCL: now also J2.1
- net SDA: now also J1.1
Routing:
- net MOSI: track 9.52 -> 7.12 mm
- net GND: track 221.7 -> 219.3 mm
- net SCK: track 24.8 -> 23.8 mm
- net SDA: track 41.3 -> 41.9 mm
Changed lines of the file:
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@@
 <element name="U$2" library="fab" package="SJFAB" value="SOLDER_JUMPER" x="7.9375" y="6.985" rot="R180"/>
 <element name="JP3" library="SparkFun" package="1X06-KIT" value="FTDI Basic" x="47.8455125" y="15.078259375" rot="R270"/>
-<element name="J1" library="SparkFun-Connectors" package="1X01NS-KIT" value="" x="19.05" y="3.81"/>
-<element name="J2" library="SparkFun-Connectors" package="1X01NS-KIT" value="" x="26.67" y="3.81"/>
-<element name="J3" library="SparkFun-Connectors" package="1X01NS-KIT" value="" x="13.335" y="6.35"/>
-<element name="J4" library="SparkFun-Connectors" package="1X01NS-KIT" value="" x="13.335" y="8.89"/>
+<element name="J1" library="SparkFun-Connectors" package="1X01" value="" x="34.925" y="23.495"/>
+<element name="J2" library="SparkFun-Connectors" package="1X01" value="" x="34.925" y="20.955"/>
 </elements>
 <signals>
@@
 <vertex x="50.165" y="48.26"/>
 </polygon>
-<contactref element="J4" pad="1"/>
-<wire x1="13.335" y1="8.89" x2="15.5225" y2="8.89" width="0.4064" layer="1"/>
-<wire x1="15.5225" y1="8.89" x2="15.5225" y2="9.04" width="0.4064" layer="1"/>
 <contactref element="R1" pad="2"/>
 <wire x1="45.505040625" y1="27.519959375" x2="45.72" y2="27.519959375" width="0.254" layer="1"/>
@@
 <wire x1="5.92034375" y1="16.4815375" x2="5.98" y2="16.4815375" width="0.4064" layer="1"/>
 <wire x1="5.98" y1="16.4815375" x2="5.98" y2="18" width="0.4064" layer="1"/>
+<wire x1="5.92034375" y1="16.25" x2="5.715" y2="16.25" width="0.4064" layer="1"/>
+<wire x1="5.715" y1="16.25" x2="5.715" y2="17.78" width="0.4064" layer="1"/>
+<wire x1="5.715" y1="17.78" x2="3.978934375" y2="17.78" width="0.254" layer="1"/>
+<wire x1="3.978934375" y1="17.78" x2="3.978934375" y2="17.9239125" width="0.254" layer="1"/>
+<wire x1="3.978934375" y1="17.9239125" x2="3.863603125" y2="17.9239125" width="0.254" layer="1"/>
+<wire x1="3.863603125" y1="17.9239125" x2="3.863603125" y2="13.53909375" width="0.254" layer="1"/>
+<wire x1="3.863603125" y1="13.53909375" x2="7.13" y2="13.53909375" width="0.4064" layer="1"/>
+<wire x1="7.13" y1="13.53909375" x2="7.13" y2="13.5" width="0.4064" layer="1"/>
 <wire x1="43.12525" y1="25.619959375" x2="41.72525" y2="26.019959375" width="0" layer="19" extent="1-1"/>
 <wire x1="12.0874" y1="15.6" x2="12.0856125" y2="15.6017875" width="0" layer="19" extent="1-1"/>
@@
 <wire x1="45.41265625" y1="35.9451125" x2="47.88" y2="36.15990625" width="0" layer="19" extent="1-1"/>
 <wire x1="40.88" y1="21.35" x2="40.88" y2="24.25" width="0" layer="19" extent="1-1"/>
-<wire x1="5.92034375" y1="16.25" x2="5.715" y2="16.25" width="0.4064" layer="1"/>
-<wire x1="5.715" y1="16.25" x2="5.715" y2="17.78" width="0.4064" layer="1"/>
-<wire x1="5.715" y1="17.78" x2="3.978934375" y2="17.78" width="0.254" layer="1"/>
-<wire x1="3.978934375" y1="17.78" x2="3.978934375" y2="17.9239125" width="0.254" layer="1"/>
-<wire x1="3.978934375" y1="17.9239125" x2="3.863603125" y2="17.9239125" width="0.254" layer="1"/>
-<wire x1="3.863603125" y1="17.9239125" x2="3.863603125" y2="13.53909375" width="0.254" layer="1"/>
-<wire x1="3.863603125" y1="13.53909375" x2="7.13" y2="13.53909375" width="0.4064" layer="1"/>
-<wire x1="7.13" y1="13.53909375" x2="7.13" y2="13.5" width="0.4064" layer="1"/>
 </signal>
 <signal name="N$1">
@@
 <wire x1="27.379040625" y1="30.752546875" x2="25.49419375" y2="28.8677" width="0.508" layer="1"/>
 <wire x1="38.63" y1="24.75" x2="38.63" y2="24.25" width="0.508" layer="1"/>
-<wire x1="38.63" y1="21.25" x2="28.13" y2="21.25" width="0.508" layer="1"/>
+<wire x1="38.63" y1="21.25" x2="34.925" y2="21.25" width="0.508" layer="1"/>
+<wire x1="34.925" y1="21.25" x2="28.13" y2="21.25" width="0.508" layer="1"/>
 <wire x1="28.13" y1="21.25" x2="25.49419375" y2="23.88580625" width="0.508" layer="1"/>
 <wire x1="39.63" y1="25.75" x2="38.63" y2="24.75" width="0.508" layer="1"/>
@@
 <wire x1="27.811828125" y1="31.897421875" x2="27.811828125" y2="31.185334375" width="0.2286" layer="1"/>
 <wire x1="27.811828125" y1="31.185334375" x2="27.379040625" y2="30.752546875" width="0.2286" layer="1"/>
-<wire x1="38.63" y1="21.25" x2="38.63" y2="24.25" width="0" layer="19" extent="1-1"/>
+<contactref element="J2" pad="1"/>
+<wire x1="34.925" y1="20.955" x2="34.925" y2="21.25" width="0.3048" layer="1"/>
 <wire x1="27.80950625" y1="31.89974375" x2="27.811828125" y2="31.897421875" width="0" layer="19" extent="1-1"/>
 <wire x1="22.13" y1="23.25" x2="24.88" y2="23.2716125" width="0" layer="19" extent="1-1"/>
+<wire x1="38.63" y1="21.25" x2="38.63" y2="24.25" width="0" layer="19" extent="1-1"/>
 </signal>
 <signal name="SDA">
@@
 <wire x1="42.62525" y1="23.57525" x2="41.91" y2="22.86" width="0.2286" layer="1"/>
 <wire x1="31.13" y1="22.845" x2="31.115" y2="22.86" width="0.508" layer="1"/>
-<wire x1="31.115" y1="22.86" x2="41.91" y2="22.86" width="0.508" layer="1"/>
+<wire x1="31.115" y1="22.86" x2="34.925" y2="22.86" width="0.508" layer="1"/>
+<wire x1="34.925" y1="22.86" x2="41.91" y2="22.86" width="0.508" layer="1"/>
 <wire x1="31.115" y1="22.86" x2="28.575" y2="22.86" width="0.508" layer="1"/>
 <wire x1="28.575" y1="22.86" x2="26.993965625" y2="24.45215625" width="0.508" layer="1"/>
@@
 <wire x1="28.30895625" y1="31.89919375" x2="28.30895625" y2="31.1906125" width="0.2286" layer="1"/>
 <wire x1="28.30895625" y1="31.1906125" x2="28.57989375" y2="30.919675" width="0.2286" layer="1"/>
+<contactref element="J1" pad="1"/>
+<wire x1="34.925" y1="23.495" x2="34.925" y2="22.86" width="0.3048" layer="1"/>
 <wire x1="28.30895625" y1="31.89919375" x2="28.30950625" y2="31.89974375" width="0" layer="19" extent="1-1"/>
 <wire x1="31.13" y1="19.75" x2="31.13" y2="22.845" width="0" layer="19" extent="1-1"/>
@@
 <wire x1="18.13" y1="41.25" x2="16.88" y2="42.5" width="0.508" layer="1"/>
 <wire x1="16.88" y1="42.5" x2="13.052" y2="42.5" width="0.508" layer="1"/>
-<wire x1="21.2375" y1="9.04" x2="21.1975" y2="9" width="0.508" layer="1"/>
 <wire x1="23.38" y1="4.75" x2="23.38" y2="2.75" width="0.508" layer="1"/>
 <wire x1="23.38" y1="2.75" x2="22.245" y2="1.615" width="0.508" layer="1"/>
@@
 <wire x1="12.38" y1="44.5" x2="13.052" y2="43.828" width="0.508" layer="1"/>
 <wire x1="13.052" y1="43.828" x2="13.052" y2="42.5" width="0.508" layer="1"/>
-<wire x1="19.26545625" y1="5.49954375" x2="19.26545625" y2="8.38545625" width="0.3048" layer="1"/>
-<wire x1="19.541321875" y1="5.223678125" x2="23.0260625" y2="5.223678125" width="0.3048" layer="1"/>
-<wire x1="19.26545625" y1="8.38545625" x2="19.88" y2="9" width="0.3048" layer="1"/>
-<wire x1="19.88" y1="9" x2="21.1975" y2="9" width="0.3048" layer="1"/>
-<wire x1="19.541321875" y1="5.223678125" x2="19.26545625" y2="5.49954375" width="0.3048" layer="1"/>
-<wire x1="23.0260625" y1="5.223678125" x2="23.0260625" y2="5.1039375" width="0.3048" layer="1"/>
-<wire x1="23.0260625" y1="5.1039375" x2="23.38" y2="4.75" width="0.3048" layer="1"/>
 <wire x1="15.98" y1="20.2926" x2="15.98" y2="27.13596875" width="0.3048" layer="1"/>
 <wire x1="15.98" y1="27.13596875" x2="15.98294375" y2="27.1389125" width="0.3048" layer="1"/>
+<wire x1="21.2375" y1="9.04" x2="19.835" y2="9.04" width="0.3048" layer="1"/>
+<wire x1="19.835" y1="9.04" x2="19.05" y2="8.255" width="0.3048" layer="1"/>
+<wire x1="19.05" y1="8.255" x2="19.05" y2="5.715" width="0.3048" layer="1"/>
+<wire x1="19.05" y1="5.715" x2="19.685" y2="5.08" width="0.3048" layer="1"/>
+<wire x1="19.685" y1="5.08" x2="23.05" y2="5.08" width="0.3048" layer="1"/>
+<wire x1="23.05" y1="5.08" x2="23.38" y2="4.75" width="0.3048" layer="1"/>
 </signal>
 <signal name="SCK">
@@
 <wire x1="21.09" y1="13.2" x2="22.225" y2="12.065" width="0.3048" layer="1"/>
 <wire x1="22.225" y1="12.065" x2="24.13" y2="10.16" width="0.508" layer="1"/>
-<contactref element="J2" pad="1"/>
-<wire x1="26.67" y1="3.81" x2="26.67" y2="4.75" width="0.4064" layer="1"/>
 </signal>
 <signal name="MISO">
@@
 <wire x1="19.05" y1="3.81" x2="21.0875" y2="3.81" width="0.3048" layer="1"/>
 <wire x1="21.0875" y1="3.81" x2="21.2375" y2="3.96" width="0.3048" layer="1"/>
-<contactref element="J1" pad="1"/>
 </signal>
 <signal name="MOSI">
@@
 <wire x1="17.5639875" y1="7.4039875" x2="16.51" y2="6.35" width="0.3048" layer="1"/>
 <wire x1="16.51" y1="6.35" x2="15.6725" y2="6.35" width="0.3048" layer="1"/>
-<wire x1="15.6725" y1="6.35" x2="15.5225" y2="6.5" width="0.3048" layer="1"/>
-<contactref element="J3" pad="1"/>
-<wire x1="13.335" y1="6.35" x2="15.5225" y2="6.35" width="0.4064" layer="1"/>
 <wire x1="15.5225" y1="6.35" x2="15.5225" y2="6.5" width="0.4064" layer="1"/>
+<wire x1="15.5225" y1="6.35" x2="15.6725" y2="6.35" width="0" layer="19" extent="1-1"/>
 </signal>
 <signal name="TXO">
