File: PCB/9DofImu.sch (EAGLE design)
At the start: 37 parts, among them U1 ATMEGA328, U2 ITG-3200, U3 LSM303

Commit message: upadted pcb
Parts:
- added JP3: FTDI Basic, SparkFun:ARDUINO_SERIAL_PROGRAMSMD
Other:
- moved on the sheet: JP2, R1, R10, R11, R12, R13, R14, R2, R5, R7
Changed lines of the file:
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@@
 <part name="JP2" library="SparkFun" deviceset="ARDUINO_SERIAL_PROGRAM" device="SMD" value="FTDI Basic"/>
 <part name="U$2" library="fab" deviceset="SOLDER_JUMPER" device=""/>
+<part name="JP3" library="SparkFun" deviceset="ARDUINO_SERIAL_PROGRAM" device="SMD" value="FTDI Basic"/>
 </parts>
 <sheets>
@@
 <instance part="GND6" gate="1" x="396.24" y="48.26"/>
 <instance part="P+6" gate="G$1" x="388.62" y="76.2"/>
-<instance part="R1" gate="G$1" x="210.82" y="114.3"/>
-<instance part="R2" gate="G$1" x="210.82" y="106.68"/>
-<instance part="R5" gate="G$1" x="210.82" y="99.06"/>
+<instance part="R1" gate="G$1" x="195.58" y="114.3"/>
+<instance part="R2" gate="G$1" x="195.58" y="106.68"/>
+<instance part="R5" gate="G$1" x="195.58" y="99.06"/>
 <instance part="FRAME2" gate="G$1" x="167.64" y="-40.64"/>
 <instance part="FRAME2" gate="G$2" x="314.96" y="-40.64"/>
-<instance part="R7" gate="G$1" x="226.06" y="114.3"/>
-<instance part="R10" gate="G$1" x="226.06" y="106.68"/>
-<instance part="R11" gate="G$1" x="226.06" y="99.06"/>
-<instance part="R12" gate="G$1" x="241.3" y="114.3"/>
-<instance part="R13" gate="G$1" x="241.3" y="106.68"/>
-<instance part="R14" gate="G$1" x="241.3" y="99.06"/>
-<instance part="JP2" gate="G$1" x="274.32" y="104.14"/>
+<instance part="R7" gate="G$1" x="210.82" y="114.3"/>
+<instance part="R10" gate="G$1" x="210.82" y="106.68"/>
+<instance part="R11" gate="G$1" x="210.82" y="99.06"/>
+<instance part="R12" gate="G$1" x="226.06" y="114.3"/>
+<instance part="R13" gate="G$1" x="226.06" y="106.68"/>
+<instance part="R14" gate="G$1" x="226.06" y="99.06"/>
+<instance part="JP2" gate="G$1" x="259.08" y="104.14"/>
+<instance part="JP3" gate="G$1" x="281.94" y="104.14"/>
 </instances>
 <busses>

Commit message: pcb updates
Parts:
- added J1, J2, J3, J4: (no value), SparkFun-Connectors:M01NOSILK-KIT
- JP1, JP2, JP3: device SparkFun:ARDUINO_SERIAL_PROGRAMSMD -> SparkFun:ARDUINO_SERIAL_PROGRAMPTH-KIT
Connections:
- net GND: now also J4.1, R1.2
- net MISO: now also J1.1
- net MOSI: now also J3.1
- net SCK: now also J2.1

Commit message: i2c pin headers
Parts:
- removed J3, J4: (no value), SparkFun-Connectors:M01NOSILK-KIT
- J1, J2: device SparkFun-Connectors:M01NOSILK-KIT -> SparkFun-Connectors:M01PTH
Connections:
- net GND: no longer J4.1
- net MISO: no longer J1.1
- net MOSI: no longer J3.1
- net SCK: no longer J2.1
- net SCL: now also J2.1
- net SDA: now also J1.1
Other:
- moved on the sheet: J1, J2
Changed lines of the file:
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@@
 <grid distance="0.1" unitdist="inch" unit="inch" style="lines" multiple="1" display="no" altdistance="0.01" altunitdist="inch" altunit="inch"/>
 <layers>
-<layer number="1" name="Top" color="4" fill="1" visible="yes" active="no"/>
-<layer number="2" name="Route2" color="1" fill="3" visible="yes" active="no"/>
-<layer number="3" name="Route3" color="4" fill="3" visible="yes" active="no"/>
-<layer number="14" name="Route14" color="1" fill="6" visible="yes" active="no"/>
-<layer number="15" name="Route15" color="4" fill="6" visible="yes" active="no"/>
-<layer number="16" name="Bottom" color="1" fill="1" visible="yes" active="no"/>
-<layer number="17" name="Pads" color="2" fill="1" visible="yes" active="no"/>
-<layer number="18" name="Vias" color="2" fill="1" visible="yes" active="no"/>
-<layer number="19" name="Unrouted" color="6" fill="1" visible="yes" active="no"/>
-<layer number="20" name="Dimension" color="15" fill="1" visible="yes" active="no"/>
-<layer number="21" name="tPlace" color="7" fill="1" visible="yes" active="no"/>
-<layer number="22" name="bPlace" color="7" fill="1" visible="yes" active="no"/>
-<layer number="23" name="tOrigins" color="15" fill="1" visible="yes" active="no"/>
-<layer number="24" name="bOrigins" color="15" fill="1" visible="yes" active="no"/>
-<layer number="25" name="tNames" color="7" fill="1" visible="yes" active="no"/>
-<layer number="26" name="bNames" color="7" fill="1" visible="yes" active="no"/>
-<layer number="27" name="tValues" color="7" fill="1" visible="yes" active="no"/>
-<layer number="28" name="bValues" color="7" fill="1" visible="yes" active="no"/>
+<layer number="1" name="Top" color="4" fill="1" visible="no" active="no"/>
+<layer number="2" name="Route2" color="1" fill="3" visible="no" active="no"/>
+<layer number="3" name="Route3" color="4" fill="3" visible="no" active="no"/>
+<layer number="14" name="Route14" color="1" fill="6" visible="no" active="no"/>
+<layer number="15" name="Route15" color="4" fill="6" visible="no" active="no"/>
+<layer number="16" name="Bottom" color="1" fill="1" visible="no" active="no"/>
+<layer number="17" name="Pads" color="2" fill="1" visible="no" active="no"/>
+<layer number="18" name="Vias" color="2" fill="1" visible="no" active="no"/>
+<layer number="19" name="Unrouted" color="6" fill="1" visible="no" active="no"/>
+<layer number="20" name="Dimension" color="15" fill="1" visible="no" active="no"/>
+<layer number="21" name="tPlace" color="7" fill="1" visible="no" active="no"/>
+<layer number="22" name="bPlace" color="7" fill="1" visible="no" active="no"/>
+<layer number="23" name="tOrigins" color="15" fill="1" visible="no" active="no"/>
+<layer number="24" name="bOrigins" color="15" fill="1" visible="no" active="no"/>
+<layer number="25" name="tNames" color="7" fill="1" visible="no" active="no"/>
+<layer number="26" name="bNames" color="7" fill="1" visible="no" active="no"/>
+<layer number="27" name="tValues" color="7" fill="1" visible="no" active="no"/>
+<layer number="28" name="bValues" color="7" fill="1" visible="no" active="no"/>
 <layer number="29" name="tStop" color="7" fill="3" visible="no" active="no"/>
 <layer number="30" name="bStop" color="7" fill="6" visible="no" active="no"/>
@@
 <layer number="35" name="tGlue" color="7" fill="4" visible="no" active="no"/>
 <layer number="36" name="bGlue" color="7" fill="5" visible="no" active="no"/>
-<layer number="37" name="tTest" color="7" fill="1" visible="yes" active="no"/>
-<layer number="38" name="bTest" color="7" fill="1" visible="yes" active="no"/>
+<layer number="37" name="tTest" color="7" fill="1" visible="no" active="no"/>
+<layer number="38" name="bTest" color="7" fill="1" visible="no" active="no"/>
 <layer number="39" name="tKeepout" color="4" fill="11" visible="no" active="no"/>
 <layer number="40" name="bKeepout" color="1" fill="11" visible="no" active="no"/>
@@
 <layer number="44" name="Drills" color="7" fill="1" visible="no" active="no"/>
 <layer number="45" name="Holes" color="7" fill="1" visible="no" active="no"/>
-<layer number="46" name="Milling" color="3" fill="1" visible="yes" active="no"/>
-<layer number="47" name="Measures" color="7" fill="1" visible="yes" active="no"/>
-<layer number="48" name="Document" color="7" fill="1" visible="yes" active="no"/>
-<layer number="49" name="Reference" color="7" fill="1" visible="yes" active="no"/>
-<layer number="50" name="dxf" color="7" fill="1" visible="yes" active="no"/>
-<layer number="51" name="tDocu" color="7" fill="1" visible="yes" active="no"/>
-<layer number="52" name="bDocu" color="7" fill="1" visible="yes" active="no"/>
-<layer number="53" name="tGND_GNDA" color="7" fill="9" visible="yes" active="no"/>
-<layer number="54" name="bGND_GNDA" color="1" fill="9" visible="yes" active="no"/>
-<layer number="56" name="wert" color="7" fill="1" visible="yes" active="no"/>
-<layer number="57" name="tCAD" color="7" fill="1" visible="yes" active="no"/>
-<layer number="59" name="tCarbon" color="7" fill="1" visible="yes" active="no"/>
-<layer number="60" name="bCarbon" color="7" fill="1" visible="yes" active="no"/>
+<layer number="46" name="Milling" color="3" fill="1" visible="no" active="no"/>
+<layer number="47" name="Measures" color="7" fill="1" visible="no" active="no"/>
+<layer number="48" name="Document" color="7" fill="1" visible="no" active="no"/>
+<layer number="49" name="Reference" color="7" fill="1" visible="no" active="no"/>
+<layer number="50" name="dxf" color="7" fill="1" visible="no" active="no"/>
+<layer number="51" name="tDocu" color="7" fill="1" visible="no" active="no"/>
+<layer number="52" name="bDocu" color="7" fill="1" visible="no" active="no"/>
+<layer number="53" name="tGND_GNDA" color="7" fill="9" visible="no" active="no"/>
+<layer number="54" name="bGND_GNDA" color="1" fill="9" visible="no" active="no"/>
+<layer number="56" name="wert" color="7" fill="1" visible="no" active="no"/>
+<layer number="57" name="tCAD" color="7" fill="1" visible="no" active="no"/>
+<layer number="59" name="tCarbon" color="7" fill="1" visible="no" active="no"/>
+<layer number="60" name="bCarbon" color="7" fill="1" visible="no" active="no"/>
 <layer number="90" name="Modules" color="5" fill="1" visible="yes" active="yes"/>
 <layer number="91" name="Nets" color="2" fill="1" visible="yes" active="yes"/>
@@
 <part name="U$2" library="fab" deviceset="SOLDER_JUMPER" device=""/>
 <part name="JP3" library="SparkFun" deviceset="ARDUINO_SERIAL_PROGRAM" device="PTH-KIT" value="FTDI Basic"/>
-<part name="J1" library="SparkFun-Connectors" deviceset="M01" device="NOSILK-KIT"/>
-<part name="J2" library="SparkFun-Connectors" deviceset="M01" device="NOSILK-KIT"/>
-<part name="J3" library="SparkFun-Connectors" deviceset="M01" device="NOSILK-KIT"/>
-<part name="J4" library="SparkFun-Connectors" deviceset="M01" device="NOSILK-KIT"/>
 <part name="GND7" library="SparkFun" deviceset="GND" device=""/>
+<part name="J1" library="SparkFun-Connectors" deviceset="M01" device="PTH"/>
+<part name="J2" library="SparkFun-Connectors" deviceset="M01" device="PTH"/>
 </parts>
 <sheets>
@@
 <instance part="C11" gate="G$1" x="139.7" y="144.78"/>
 <instance part="U$2" gate="G$1" x="96.52" y="137.16" rot="R90"/>
-<instance part="J1" gate="G$1" x="55.88" y="132.08"/>
-<instance part="J2" gate="G$1" x="55.88" y="129.54"/>
-<instance part="J3" gate="G$1" x="104.14" y="129.54" rot="R180"/>
-<instance part="J4" gate="G$1" x="99.06" y="124.46" rot="R180"/>
+<instance part="J1" gate="G$1" x="20.32" y="121.92"/>
+<instance part="J2" gate="G$1" x="20.32" y="111.76"/>
 </instances>
 <busses>
@@
 <wire x1="83.82" y1="127" x2="91.44" y2="127" width="0.1524" layer="91"/>
 <pinref part="GND17" gate="1" pin="GND"/>
-<wire x1="91.44" y1="127" x2="91.44" y2="124.46" width="0.1524" layer="91"/>
-<pinref part="J4" gate="G$1" pin="1"/>
-<wire x1="91.44" y1="124.46" x2="91.44" y2="121.92" width="0.1524" layer="91"/>
-<junction x="91.44" y="124.46"/>
+<wire x1="91.44" y1="127" x2="91.44" y2="121.92" width="0.1524" layer="91"/>
 </segment>
 </net>
@@
 <pinref part="U1" gate="G$1" pin="PC5(ADC5/SCL)"/>
 </segment>
+<segment>
+<pinref part="J2" gate="G$1" pin="1"/>
+<wire x1="27.94" y1="111.76" x2="38.1" y2="111.76" width="0.1524" layer="91"/>
+<label x="30.48" y="111.76" size="1.778" layer="95"/>
+</segment>
 </net>
 <net name="SDA" class="0">
@@
 <label x="233.68" y="134.62" size="1.778" layer="95"/>
 <pinref part="U1" gate="G$1" pin="PC4(ADC4/SDA)"/>
+</segment>
+<segment>
+<pinref part="J1" gate="G$1" pin="1"/>
+<wire x1="27.94" y1="121.92" x2="38.1" y2="121.92" width="0.1524" layer="91"/>
+<label x="30.48" y="121.92" size="1.778" layer="95"/>
 </segment>
 </net>
@@
 <wire x1="76.2" y1="129.54" x2="63.5" y2="129.54" width="0.1524" layer="91"/>
 <label x="63.5" y="129.54" size="1.778" layer="95"/>
-<pinref part="J2" gate="G$1" pin="1"/>
 </segment>
 </net>
@@
 <wire x1="76.2" y1="132.08" x2="63.5" y2="132.08" width="0.1524" layer="91"/>
 <label x="63.5" y="132.08" size="1.778" layer="95"/>
-<pinref part="J1" gate="G$1" pin="1"/>
 </segment>
 </net>
@@
 <wire x1="83.82" y1="129.54" x2="96.52" y2="129.54" width="0.1524" layer="91"/>
 <label x="91.44" y="129.54" size="1.778" layer="95"/>
-<pinref part="J3" gate="G$1" pin="1"/>
-</segment>
-</net>
+</segment>
+</net>
